File: PCB/SMP_back/SysMonPro.kicad_sch (KiCad schematic)
At the start: 20 parts, among them J8 V3-, J9 V3+

Commit message: enlarged hole
Parts:
- C1, C2: value (none) -> 22p; footprint (none) -> Capacitor_SMD:C_0805_2012Metric_Pad1.18x1.45mm_HandSolder
- C3: value (none) -> 1u; footprint (none) -> Capacitor_SMD:C_0805_2012Metric_Pad1.18x1.45mm_HandSolder
- J1: value (none) -> V0+; footprint MountingHole:MountingHole_3.2mm_M3_Pad_Via -> MountingHole:MountingHole_4.3mm_M4_Pad_Via
- J2: value (none) -> V1+; footprint MountingHole:MountingHole_3.2mm_M3_Pad_Via -> MountingHole:MountingHole_4.3mm_M4_Pad_Via
- J3: value (none) -> V2+; footprint MountingHole:MountingHole_3.2mm_M3_Pad_Via -> MountingHole:MountingHole_4.3mm_M4_Pad_Via
- J4: value (none) -> Conn_02x03_Counter_Clockwise; footprint (none) -> Connector_PinSocket_2.54mm:PinSocket_2x03_P2.54mm_Vertical
- J5: value (none) -> V0-; footprint MountingHole:MountingHole_3.2mm_M3_Pad_Via -> MountingHole:MountingHole_4.3mm_M4_Pad_Via
- J6: value (none) -> V1-; footprint MountingHole:MountingHole_3.2mm_M3_Pad_Via -> MountingHole:MountingHole_4.3mm_M4_Pad_Via
- J7: value (none) -> V2-; footprint MountingHole:MountingHole_3.2mm_M3_Pad_Via -> MountingHole:MountingHole_4.3mm_M4_Pad_Via
- J8, J9: footprint MountingHole:MountingHole_3.2mm_M3_Pad_Via -> MountingHole:MountingHole_4.3mm_M4_Pad_Via
- P1: value (none) -> USB_C_Plug_USB2.0; footprint (none) -> Connector_USB:USB_C_Receptacle_Palconn_UTC16-G
- R1, R2: value (none) -> 22; footprint (none) -> Resistor_SMD:R_0805_2012Metric_Pad1.20x1.40mm_HandSolder
- R3, R4: value (none) -> 5k1; footprint (none) -> Resistor_SMD:R_0805_2012Metric_Pad1.20x1.40mm_HandSolder
- SW1: value (none) -> SW_Push; footprint (none) -> Button_Switch_SMD:SW_SPST_SKQG_WithStem
- U1: value (none) -> ATmega32U4-AU; footprint (none) -> Package_QFP:TQFP-44_10x10mm_P0.8mm
- Y1: value (none) -> XTAL; footprint (none) -> Crystal:Crystal_SMD_3225-4Pin_3.2x2.5mm_HandSoldering
